Commit message: - Fixed niryo gripper joint axes - Improved some block tooltips

File: assets/models/niryo_robot_description/urdf/ned/niryo_ned_gripper.urdf.xacro (robot description, xacro)
@@ -92,5 +92,5 @@
         <parent link="base_gripper_1"/>
         <child link="mors_1"/>
-        <axis xyz="0 1 0"/>
+        <axis xyz="0 0 1"/>
         <limit lower="-0.01"
                upper="0.01"
@@ -136,5 +136,5 @@
         <parent link="base_gripper_1"/>
         <child link="mors_2"/>
-        <axis xyz="0 -1 0"/>
+        <axis xyz="0 0 -1"/>
         <limit lower="-0.01"
                upper="0.01"
