Commit message: - Added robotiq 2 finger and 3 finger grippers - Switched to 2 finger gripper for sawyer - rewrote part of the robot initialization - new robots now only need to define at which links the robot and the hand starts - added option to invert open and close (required for robotiq 2f gripper) - added onLoadComplete callback to robot (called when all rendering is done)

File: assets/models/sawyer_description/urdf/sawyer_rocksi.urdf.xacro (robot description, xacro)
@@ -1,402 +1,21 @@
 <?xml version="1.0" ?>
 <robot name="sawyer" xmlns:xacro="http://www.ros.org/wiki/xacro">
-  <material name="black">
-    <color rgba="0 0 0 1"/>
-  </material>
-  <material name="darkgray">
-    <color rgba=".2 .2 .2 1"/>
-  </material>
-  <material name="darkred">
-    <color rgba=".5 .1 .1 1"/>
-  </material>
-  <material name="sawyer_red">
-    <color rgba=".5 .1 .1 1"/>
-  </material>
-  <material name="sawyer_gray">
-    <color rgba="0.75294 0.75294 0.75294 1"/>
-  </material>
-  <link name="base"/>
-  <link name="torso">
-    <visual>
-      <origin rpy="0 0 0" xyz="0 0 0"/>
-      <geometry>
-        <box size="0.001 0.001 0.001"/>
-      </geometry>
-      <material name="darkgray">
-        <color rgba=".2 .2 .2 1"/>
-      </material>
-    </visual>
-  </link>
-  <joint name="right_arm_mount" type="fixed">
-    <origin rpy="0 0 0" xyz="0.0 0.0 0.0"/>
-    <parent link="base"/>
-    <child link="right_arm_base_link"/>
-  </joint>
-  <joint name="torso_t0" type="fixed">
-    <origin rpy="0 0 0" xyz="0 0 0"/>
-    <parent link="base"/>
-    <child link="torso"/>
-  </joint>
-  <link name="right_arm_base_link">
-    <inertial>
-      <origin rpy="0 0 0" xyz="-0.0006241 -2.8025E-05 0.065404"/>
-      <mass value="2.0687"/>
-      <inertia ixx="0.0067599" ixy="-4.2024E-05" ixz="-6.1904E-07" iyy="0.0067877" iyz="1.5888E-05" izz="0.0074031"/>
-    </inertial>
-    <visual>
-      <origin rpy="0 0 0" xyz="0 0 0"/>
-      <geometry>
-        <mesh filename="package://sawyer_description/meshes/sawyer_pv/base.DAE"/>
-      </geometry>
-      <material name="sawyer_red"/>
-    </visual>
-    <collision>
-      <origin rpy="0 0 0" xyz="0 0 0.12"/>
-      <geometry>
-        <cylinder length="0.24" radius="0.08"/>
-      </geometry>
-    </collision>
-  </link>
-  <link name="right_l0">
-    <inertial>
-      <origin rpy="0 0 0" xyz="0.024366 0.010969 0.14363"/>
-      <mass value="5.3213"/>
-      <inertia ixx="0.053314" ixy="0.0047093" ixz="0.011734" iyy="0.057902" iyz="0.0080179" izz="0.023659"/>
-    </inertial>
-    <visual>
-      <origin rpy="0 0 0" xyz="0 0 0"/>
-      <geometry>
-        <mesh filename="package://sawyer_description/meshes/sawyer_mp3/l0.DAE"/>
-      </geometry>
-      <material name="sawyer_red"/>
-    </visual>
-    <collision>
-      <origin rpy="0 0 0" xyz="0.08 0 0.23"/>
-      <geometry>
-        <sphere radius="0.07"/>
-      </geometry>
-    </collision>
-  </link>
-  <joint name="right_j0" type="revolute">
-    <origin rpy="0 0 0" xyz="0 0 0.08"/>
-    <parent link="right_arm_base_link"/>
-    <child link="right_l0"/>
-    <axis xyz="0 0 1"/>
-    <limit effort="80.0" lower="-3.0503" upper="3.0503" velocity="1.74"/>
-    <dynamics damping="10.0" friction="5.0"/>
-  </joint>
-  <link name="head">
-    <inertial>
-      <origin rpy="0 0 0" xyz="0.0053207 -2.6549E-05 0.1021"/>
-      <mass value="1.5795"/>
-      <inertia ixx="0.011833" ixy="-4.4669E-06" ixz="4.9425E-05" iyy="0.0082709" iyz="4.2124E-07" izz="0.0049661"/>
-    </inertial>
-    <visual>
-      <origin rpy="0 0 0" xyz="0 0 0"/>
-      <geometry>
-        <mesh filename="package://sawyer_description/meshes/sawyer_pv/head.DAE"/>
-      </geometry>
-      <material name="sawyer_red"/>
-    </visual>
-    <collision>
-      <origin rpy="0 0 0" xyz="0 0 0.08"/>
-      <geometry>
-        <sphere radius="0.18"/>
-      </geometry>
-    </collision>
-  </link>
-  <joint name="head_pan" type="revolute">
-    <origin rpy="0 0 0" xyz="0 0 0.2965"/>
-    <parent link="right_l0"/>
-    <child link="head"/>
-    <axis xyz="0 0 1"/>
-    <limit effort="8" lower="-5.0952" upper="0.9064" velocity="1.8"/>
-    <dynamics damping="1.0" friction="0.5"/>
-  </joint>
-  <link name="right_torso_itb_l">
-  </link>
-  <joint name="right_torso_itb_j" type="fixed">
-    <origin rpy="0 -1.57079632679 0" xyz="-.055 0 .22"/>
-    <parent link="right_l0"/>
-    <child link="right_torso_itb_l"/>
-    <axis xyz="0 0 1"/>
-  </joint>
-  <link name="right_l1">
-    <inertial>
-      <origin rpy="0 0 0" xyz="-0.0030849 -0.026811 0.092521"/>
-      <mass value="4.505"/>
-      <inertia ixx="0.022398" ixy="-0.00023986" ixz="-0.00029362" iyy="0.014613" iyz="-0.0060875" izz="0.017295"/>
-    </inertial>
-    <visual>
-      <origin rpy="0 0 0" xyz="0 0 0"/>
-      <geometry>
-        <mesh filename="package://sawyer_description/meshes/sawyer_mp3/l1.DAE"/>
-      </geometry>
-      <material name="sawyer_red"/>
-    </visual>
-    <collision>
-      <origin rpy="0 0 0" xyz="0 0 0.1225"/>
-      <geometry>
-        <sphere radius="0.07"/>
-      </geometry>
-    </collision>
-  </link>
-  <joint name="right_j1" type="revolute">
-    <origin rpy="-1.57079632679 1.57079632679 0" xyz="0.081 0.05 0.237"/>
-    <parent link="right_l0"/>
-    <child link="right_l1"/>
-    <axis xyz="0 0 1"/>
-    <limit effort="80.0" lower="-3.8095" upper="2.2736" velocity="1.328"/>
-    <dynamics damping="5.0" friction="2.0"/>
-  </joint>
-  <link name="right_l2">
-    <inertial>
-      <origin rpy="0 0 0" xyz="-0.00016044 -0.014967 0.13582"/>
-      <mass value="1.745"/>
-      <inertia ixx="0.025506" ixy="4.4101E-06" ixz="1.4955E-05" iyy="0.0253" iyz="-0.0033204" izz="0.0034179"/>
-    </inertial>
-    <visual>
-      <origin rpy="0 0 0" xyz="0 0 0"/>
-      <geometry>
-        <mesh filename="package://sawyer_description/meshes/sawyer_pv/l2.DAE"/>
-      </geometry>
-      <material name="sawyer_red"/>
-    </visual>
-    <collision>
-      <origin rpy="0 0 0" xyz="0 0 0.08"/>
-      <geometry>
-        <cylinder length="0.34" radius="0.06"/>
-      </geometry>
-    </collision>
-  </link>
-  <joint name="right_j2" type="revolute">
-    <origin rpy="1.57079632679 0 0" xyz="0 -0.14 0.1425"/>
-    <parent link="right_l1"/>
-    <child link="right_l2"/>
-    <axis xyz="0 0 1"/>
-    <limit effort="40.0" lower="-3.0426" upper="3.0426" velocity="1.957"/>
-    <dynamics damping="5.0" friction="2.0"/>
-  </joint>
-  <link name="right_l3">
-    <inertial>
-      <origin rpy="0 0 0" xyz="-0.0048135 -0.0281 -0.084154"/>
-      <mass value="2.5097"/>
-      <inertia ixx="0.01016" ixy="-9.7452E-06" ixz="0.00026624" iyy="0.0065685" iyz="0.0030316" izz="0.0069078"/>
-    </inertial>
-    <visual>
-      <origin rpy="0 0 0" xyz="0 0 0"/>
-      <geometry>
-        <mesh filename="package://sawyer_description/meshes/sawyer_pv/l3.DAE"/>
-      </geometry>
-      <material name="sawyer_red"/>
-    </visual>
-    <collision>
-      <origin rpy="0 0 0" xyz="0 -0.01 -0.12"/>
-      <geometry>
-        <sphere radius="0.06"/>
-      </geometry>
-    </collision>
-  </link>
-  <joint name="right_j3" type="revolute">
-    <origin rpy="-1.57079632679 0 0" xyz="0 -0.042 0.26"/>
-    <parent link="right_l2"/>
-    <child link="right_l3"/>
-    <axis xyz="0 0 1"/>
-    <limit effort="40.0" lower="-3.0439" upper="3.0439" velocity="1.957"/>
-    <dynamics damping="1.0" friction="0.5"/>
-  </joint>
-  <link name="right_l4">
-    <inertial>
-      <origin rpy="0 0 0" xyz="-0.0018844 0.0069001 0.1341"/>
-      <mass value="1.1136"/>
-      <inertia ixx="0.013557" ixy="1.8109E-05" ixz="0.00013523" iyy="0.013555" iyz="0.0010561" izz="0.0013658"/>
-    </inertial>
-    <visual>
-      <origin rpy="0 0 0" xyz="0 0 0"/>
-      <geometry>
-        <mesh filename="package://sawyer_description/meshes/sawyer_pv/l4.DAE"/>
-      </geometry>
-      <material name="sawyer_red"/>
-    </visual>
-    <collision>
-      <origin rpy="0 0 0" xyz="0 0 0.11"/>
-      <geometry>
-        <cylinder length="0.30" radius="0.045"/>
-      </geometry>
-    </collision>
-  </link>
-  <joint name="right_j4" type="revolute">
-    <origin rpy="1.57079632679 0 0" xyz="0 -0.125 -0.1265"/>
-    <parent link="right_l3"/>
-    <child link="right_l4"/>
-    <axis xyz="0 0 1"/>
-    <limit effort="9.0" lower="-2.9761" upper="2.9761" velocity="3.485"/>
-    <dynamics damping="2.0" friction="1.0"/>
-  </joint>
-  <link name="right_arm_itb_l">
-  </link>
-  <joint name="right_arm_itb_j" type="fixed">
-    <origin rpy="0 -1.57079632679 0" xyz="-.055 0 .075"/>
-    <parent link="right_l4"/>
-    <child link="right_arm_itb_l"/>
-    <axis xyz="0 0 1"/>
-  </joint>
-  <link name="right_l5">
-    <inertial>
-      <origin rpy="0 0 0" xyz="0.0061133 -0.023697 0.076416"/>
-      <mass value="1.5625"/>
-      <inertia ixx="0.0047328" ixy="0.00011526" ixz="4.6269E-05" iyy="0.0029676" iyz="-0.0011557" izz="0.0031762"/>
-    </inertial>
-    <visual>
-      <origin rpy="0 0 0" xyz="0 0 0"/>
-      <geometry>
-        <mesh filename="package://sawyer_description/meshes/sawyer_pv/l5.DAE"/>
-      </geometry>
-      <material name="sawyer_red"/>
-    </visual>
-    <collision>
-      <origin rpy="0 0 0" xyz="0 0 0.1"/>
-      <geometry>
-        <sphere radius="0.06"/>
-      </geometry>
-    </collision>
-  </link>
-  <joint name="right_j5" type="revolute">
-    <origin rpy="-1.57079632679 0 0" xyz="0 0.031 0.275"/>
-    <parent link="right_l4"/>
-    <child link="right_l5"/>
-    <axis xyz="0 0 1"/>
-    <limit effort="9.0" lower="-2.9761" upper="2.9761" velocity="3.485"/>
-    <dynamics damping="1.0" friction="0.5"/>
-  </joint>
-  <link name="right_hand_camera_l"/>
-  <joint name="right_hand_camera_j" type="fixed">
-    <origin rpy="0 1.57079632679 0" xyz="0.039552 -0.033 0.0695"/>
-    <parent link="right_l5"/>
-    <child link="right_hand_camera_j"/>
-    <axis xyz="0 0 0"/>
-  </joint>
-  <link name="right_wrist_l"/>
-  <joint name="right_wrist_j" type="fixed">
-    <origin rpy="1.57079632679 0 0" xyz="0 0 0.10541"/>
-    <parent link="right_l5"/>
-    <child link="right_wrist_l"/>
-    <axis xyz="0 0 0"/>
-  </joint>
-  <link name="right_l6">
-    <inertial>
-      <origin rpy="0 0 0" xyz="-8.0726E-06 0.0085838 -0.0049566"/>
-      <mass value="0.3292"/>
-      <inertia ixx="0.00031105" ixy="1.4771E-06" ixz="-3.7074E-07" iyy="0.00021549" iyz="-8.4533E-06" izz="0.00035976"/>
-    </inertial>
-    <visual>
-      <origin rpy="0 0 0" xyz="0 0 0"/>
-      <geometry>
-        <mesh filename="package://sawyer_description/meshes/sawyer_mp1/l6.DAE"/>
-      </geometry>
-      <material name="sawyer_red"/>
-    </visual>
-    <collision>
-      <origin rpy="0 0 0" xyz="0 0.015 -0.01"/>
-      <geometry>
-        <cylinder length="0.05" radius="0.055"/>
-      </geometry>
-    </collision>
-  </link>
-  <joint name="right_j6" type="revolute">
-    <origin rpy="-1.57079632679 -0.17453 3.1416" xyz="0 -0.11 0.1053"/>
-    <parent link="right_l5"/>
-    <child link="right_l6"/>
-    <axis xyz="0 0 1"/>
-    <limit effort="9.0" lower="-3.14" upper="3.14" velocity="4.545"/>
-    <dynamics damping="1.0" friction="0.5"/>
-  </joint>
-  <link name="right_hand_l">
-    <collision>
-      <origin rpy="0 0 0" xyz="0 0 0.02"/>
-      <geometry>
-        <cylinder length="0.03" radius="0.035"/>
-      </geometry>
-    </collision>
-    <inertial>
-      <origin rpy="0 0 0" xyz="0 0.1 0"/>
-      <mass value="0.01"/>
-      <inertia ixx="0.01" ixy="0.01" ixz="0.01" iyy="0.01" iyz="0.01" izz="0.01"/>
-  </inertial>
-  </link>
-  <joint name="right_hand_j" type="fixed">
-    <origin rpy="0 0 1.570796" xyz="0 0 0.0245"/>
-    <axis xyz="0 0 1"/>
-    <parent link="right_l6"/>
-    <child link="right_hand_l"/>
-  </joint>
-  <link name="right_l1_2">
-    <collision>
-      <origin rpy="0 0 0" xyz="0 0 0.035"/>
-      <geometry>
-        <cylinder length="0.14" radius="0.07"/>
-      </geometry>
-    </collision>
-  </link>
-  <joint name="right_j1_2" type="fixed">
-    <origin rpy="0 0 0" xyz="0 0 0"/>
-    <parent link="right_l1"/>
-    <child link="right_l1_2"/>
-    <axis xyz="0 0 1"/>
-  </joint>
-  <link name="right_l2_2">
-    <collision>
-      <origin rpy="0 0 0" xyz="0 0 0.26"/>
-      <geometry>
-        <sphere radius="0.06"/>
-      </geometry>
-    </collision>
-  </link>
-  <joint name="right_j2_2" type="fixed">
-    <origin rpy="0 0 0" xyz="0 0 0"/>
-    <parent link="right_l2"/>
-    <child link="right_l2_2"/>
-    <axis xyz="0 0 1"/>
-  </joint>
-  <link name="right_l4_2">
-    <collision>
-      <origin rpy="0 0 0" xyz="0 0.01 0.26"/>
-      <geometry>
-        <sphere radius="0.06"/>
-      </geometry>
-    </collision>
-  </link>
-  <joint name="right_j4_2" type="fixed">
-    <origin rpy="0 0 0" xyz="0 0 0"/>
-    <parent link="right_l4"/>
-    <child link="right_l4_2"/>
-    <axis xyz="0 0 1"/>
-  </joint>
-  <link name="screen">
-    <visual>
-      <origin rpy="0 0 0" xyz="0 0 0"/>
-      <geometry>
-        <box size="0.24 0.14 0.002"/>
-      </geometry>
-      <material name="darkgray"/>
-    </visual>
-    <collision>
-      <origin rpy="0 0 0" xyz="0 0 0"/>
-      <geometry>
-        <sphere radius="0.001"/>
-      </geometry>
-    </collision>
-  </link>
-  <joint name="display_joint" type="fixed">
-    <origin rpy="1.57079632679 0 1.57079632679" xyz="0.03 0.0 0.105"/>
-    <parent link="head"/>
-    <child link="screen"/>
-  </joint>
-  <link name="head_camera_l"/>
-  <joint name="head_camera_j" type="fixed">
-    <origin rpy="-2.1293 0 -1.57079632679" xyz="0.0228027 0 0.216572"/>
-    <parent link="head"/>
-    <child link="head_camera_l"/>
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